File: kicad/replicazeron_stm/replicazeron_stm.kicad_sch (KiCad schematic)
At the start: 41 parts, among them J10 Conn_01x04_Pin, J1_Col1 Conn_01x06_Pin, J2_Thumb1 Conn_01x06_Pin, J3_Index1 Conn_01x06_Pin, J4_Mid1 Conn_01x06_Pin, J5_Ring1 Conn_01x06_Pin, J6_Pinky1 Conn_01x06_Pin, J7_Stick1 Conn_01x02_Pin, J8_LED1 Conn_01x02_Pin, J9 Conn_01x03_Pin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

Commit message: Routing PCB Version A
Other:
- company: (none) -> Demolite
- title: (none) -> Replicazeron PCB
Changed lines of the file:
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@@
 	(generator_version "9.0")
 	(paper "A4")
+	(title_block
+		(title "Replicazeron PCB")
+		(date "2026-01-17")
+		(rev "A")
+		(company "Demolite")
+	)
 	(junction
 		(at 60.96 85.09)
